File: design/open-amiga-sampler.kicad_pcb (KiCad board)
At the start: 2 copper layers, 37 x 34 mm, 19 parts, among them J1 Left, J2 Right, J3 DB25_Male, U1 ADC0820CCN, U2 MCP6002-xP

Commit message: Fixed op amp circuit
Connections:
- RV1 pad 3: GND -> Vo
Routing:
- net Vo: track 47.4 -> 53.7 mm
