File: smd-fork/open-amiga-sampler-smd.sch (KiCad schematic (older format))
At the start: 17 parts, among them J1 Left, J2 Right, J3 DB25_Male, U1 ADC0820CCN, U2 MCP6001U

Commit message: VCC improvements
changed mailn bulk bypass cap to electrolytic. moved C3 to close to U1 Vcc. tweaked Vcc traces for better path. Silkscreen++
Parts:
- C4: footprint Capacitor_Tantalum_SMD:CP_EIA-3216-18_Kemet-A_Pad1.58x1.35mm_HandSolder -> Capacitor_SMD:CP_Elec_4x5.3
Changed lines of the file:
@@
 F 0 "C4" H 8118 4096 50  0000 L CNN
 F 1 "47uf" H 8118 4005 50  0000 L CNN
-F 2 "Capacitor_Tantalum_SMD:CP_EIA-3216-18_Kemet-A_Pad1.58x1.35mm_HandSolder" H 8038 3900 50  0001 C CNN
+F 2 "Capacitor_SMD:CP_Elec_4x5.3" H 8038 3900 50  0001 C CNN
 F 3 "~" H 8000 4050 50  0001 C CNN
 	1    8000 4050
